File: pcb/prototype/RC2014_UX_MODULE.brd (EAGLE design)
At the start: 99.1 x 50.9 mm, 64 parts, among them IC1 P8X32A-D40, IC2 24LC256P, IC3 M74HC4078B1R, IC4 TPS7333QP

Commit message: pcb - production
Parts:
- removed C10, C11, C14, C15, C7, C8, C9: 100p, Seeed-OPL-Capacitor:C0805
- removed C12, C13, C16: 200p, Seeed-OPL-Capacitor:C0805
- removed C17: 100u, SparkFun:CPOL-RADIAL-100UF-25V
- removed IC4: TPS7333QP, TPS7333:P8_TEX
- added D4, D5, D6, D7: 1N4148DO35-7, diode:DO35-7
- added R6: 4k7, Seeed-OPL-Resistor-V2:R0207_7
- C6: value 100n -> 47u; device rcl:C025-025X050 -> SparkFun:CPOL-RADIAL-100UF-25V
- IC3: value M74HC4078B1R -> TPS7333QP; device ST Microelctronics_By_element14_Batch_1:DIP254P762X510-14 -> TPS7333:P8_TEX
- OSC1: value 7.3728MHz -> (none)
- R1, R10, R11, R12, R13, R14, R15, R16, R2, R3, R4, R5, R7, R8, R9: value 3k3 -> 4k7; device Seeed-OPL-Resistor-V2:R0805 -> Seeed-OPL-Resistor-V2:R0207_7
- R33, R34: value 3k3 -> 2k2; device Seeed-OPL-Resistor-V2:R0805 -> Seeed-OPL-Resistor-V2:R0207_7
- moved R17 71.1 mm to (24.3, 11.2)
- moved C6 64.8 mm to (89.7, 10.7), turned to 90 degrees
- moved IC3 29.3 mm to (72.9, 22.0), turned to 0 degrees
- moved D3 22.9 mm to (40.6, 11.0)
- moved R4 20.3 mm to (48.3, 11.0), turned to 90 degrees
- moved D2 15.2 mm to (38.1, 11.0)
- moved D1 15.2 mm to (35.6, 11.0)
- moved R1 9.35 mm to (27.9, 11.2), turned to 90 degrees
- moved R2 9.35 mm to (30.5, 11.2), turned to 90 degrees
- moved R3 9.35 mm to (33.0, 11.2), turned to 90 degrees
- moved R5 2.54 mm to (50.8, 11.0), turned to 90 degrees
- moved R8 2.54 mm to (63.5, 11.0), turned to 90 degrees
- moved C1 1.71 mm to (44.3, 18.7)
- moved C5 0.38 mm to (70.5, 15.6)
- moved R33 0.13 mm to (35.4, 43.3), turned to 90 degrees
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Connections:
- net P10 renamed N$3
- net P11 renamed N$4
- net P12 renamed N$5
- net P13 renamed N$6
- net P14 renamed N$7
- net P15 renamed N$8
- net P8 renamed N$1
- net P9 renamed N$2
- net XI renamed N$20
- removed net P0: C7.2, IC1.1, R1.2
- removed net P1: C8.2, IC1.2, R2.2
- removed net P2: C9.1, IC1.3, R3.1
- removed net P3: C10.2, IC1.4, R4.2
- removed net P4: C11.2, IC1.5, R5.2
- removed net P6: C14.2, IC1.7, R7.2
- removed net P7: C15.2, IC1.8, R8.2
- removed net PINT: C13.1, D2.C, IC1.34
- removed net PRESET: C12.2, D1.C, IC1.6
- removed net PWAIT: C16.1, D3.C, IC1.33
- new net !PINT: D6.C, IC1.34
- new net !PWAIT: D7.C, IC1.33
- new net N$10: IC1.7, R7.2
- new net N$11: IC1.6, R6.2
- new net N$12: IC1.5, R5.2
- new net N$13: IC1.4, R4.2
- new net N$14: IC1.3, R3.2
- new net N$15: IC1.2, R2.2
- new net N$19: D1.C, D2.C, D3.C, D4.C, D5.C, R17.1, R3.1
- new net N$9: IC1.8, R8.2
- net !DTR: now also IC3.8; no longer IC4.8
- net !INT: now also D6.A; no longer C13.2, D2.A
- net !IORQ: now also R8.1; no longer IC3.9
- net !M1: no longer C11.1
- net !RD: now also R7.1; no longer C15.1, R8.1
- net !RESET: no longer C12.1, D1.A
- net !WAIT_E: now also D7.A; no longer C16.2, D3.A
- net !WR: now also R6.1; no longer C14.1, R7.1
- net $GND: now also IC3.1, IC3.2, R17.2; no longer C17.2, IC3.10, IC3.11, IC3.7, IC4.1, IC4.2
- net $VCC: now also C6.1, FTDI_BASIC.VCC, IC3.5, IC3.6, IC3.7; no longer C17.1, IC4.5, IC4.6, IC4.7, R17.1
- net $VDD: now also IC3.3, IC3.4; no longer C6.1, IC3.14, IC4.3, IC4.4
- net BA0: no longer C10.1
- net BA1: now also D5.A; no longer IC3.5
- net BA2: now also D4.A; no longer IC3.4
- net BA3: now also D3.A; no longer IC3.3
- net BA4: now also D2.A; no longer IC3.12
- net BA5: now also D1.A; no longer IC3.2
- net BA6: no longer C8.1
- net BA7: no longer C7.1
- net N$16: now also IC1.1, R1.2; no longer C9.2, IC3.13, R3.2
- net RX: no longer R17.2
- net SCL: now also R34.1; no longer R33.1
- net SDA: now also R33.1; no longer R34.1
Routing:
- net P6: track 61.5 -> 0.00 mm
- net P7: track 61.5 -> 0.00 mm
- net !IORQ: track 64.0 -> 5.91 mm
- net P4: track 50.0 -> 0.00 mm
- net PINT: track 47.3 -> 0.00 mm
- net PWAIT: track 46.1 -> 0.00 mm
- net !PWAIT: track 0.00 -> 35.9 mm
- net BA0: track 46.1 -> 12.8 mm
- net !PINT: track 0.00 -> 31.2 mm
- net N$9: track 0.00 -> 29.5 mm
- net N$19: track 0.00 -> 28.5 mm
- net PRESET: track 28.3 -> 0.00 mm
- net N$11: track 0.00 -> 27.0 mm
- net N$10: track 0.00 -> 27.0 mm
- net BA7: track 33.8 -> 8.58 mm
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Other:
- outline, holes or cut-outs redrawn
- board text added: "Phillip Stevens - 2020"
- board text removed: "BLK"
- board text removed: "GRN"
- board text removed: "Phillip Stevens - 2021"
