File: pcb/prototype/RC2014_UX_MODULE.sch (EAGLE design)
At the start: 64 parts, among them IC1 P8X32A-D40, IC2 24LC256P, IC3 M74HC4078B1R, IC4 TPS7333QP

Commit message: pcb - production
Parts:
- removed C10, C11, C14, C15, C7, C8, C9: 100p, Seeed-OPL-Capacitor:CERAMIC-10NF-50V-5%-X7R(0805)
- removed C12, C13, C16: 200p, Seeed-OPL-Capacitor:CERAMIC-10NF-50V-5%-X7R(0805)
- removed C17: 100u, SparkFun:CAP_POLPTH1
- removed IC4: TPS7333QP, TPS7333:TPS7333QP
- added D4, D5, D6, D7: 1N4148DO35-7, diode:1N4148DO35-7
- added R6: 4k7, Seeed-OPL-Resistor-V2:RES-0207/7
- C6: value 100n -> 47u; device rcl:C-EU025-025X050 -> SparkFun:CAP_POLPTH1
- IC3: value M74HC4078B1R -> TPS7333QP; device ST Microelctronics_By_element14_Batch_1:M74HC4078B1R -> TPS7333:TPS7333QP
- OSC1: value 7.3728MHz -> (none)
- R1, R10, R11, R12, R13, R14, R15, R16, R2, R3, R4, R5, R7, R8, R9: value 3k3 -> 4k7; device Seeed-OPL-Resistor-V2:RES-0805 -> Seeed-OPL-Resistor-V2:RES-0207/7
- R33, R34: value 3k3 -> 2k2; device Seeed-OPL-Resistor-V2:RES-0805 -> Seeed-OPL-Resistor-V2:RES-0207/7
Connections:
- net P10 renamed N$3
- net P11 renamed N$4
- net P12 renamed N$5
- net P13 renamed N$6
- net P14 renamed N$7
- net P15 renamed N$8
- net P8 renamed N$1
- net P9 renamed N$2
- net XI renamed N$20
- removed net P0: C7.2, IC1.P0, R1.2
- removed net P1: C8.2, IC1.P1, R2.2
- removed net P2: C9.1, IC1.P2, R3.1
- removed net P3: C10.2, IC1.P3, R4.2
- removed net P4: C11.2, IC1.P4, R5.2
- removed net P6: C14.2, IC1.P6, R7.2
- removed net P7: C15.2, IC1.P7, R8.2
- removed net PINT: C13.1, D2.C, IC1.P25
- removed net PRESET: C12.2, D1.C, IC1.P5
- removed net PWAIT: C16.1, D3.C, IC1.P24
- new net !PINT: D6.C, IC1.P25
- new net !PWAIT: D7.C, IC1.P24
- new net N$10: IC1.P6, R7.2
- new net N$11: IC1.P5, R6.2
- new net N$12: IC1.P4, R5.2
- new net N$13: IC1.P3, R4.2
- new net N$14: IC1.P2, R3.2
- new net N$15: IC1.P1, R2.2
- new net N$19: D1.C, D2.C, D3.C, D4.C, D5.C, R17.1, R3.1
- new net N$9: IC1.P7, R8.2
- net !DTR: now also IC3.!RESET; no longer IC4.!RESET
- net !INT: now also D6.A; no longer C13.2, D2.A
- net !IORQ: now also R8.1; no longer IC3.E
- net !M1: no longer C11.1
- net !RD: now also R7.1; no longer C15.1, R8.1
- net !RESET: no longer C12.1, D1.A
- net !WAIT_E: now also D7.A; no longer C16.2, D3.A
- net !WR: now also R6.1; no longer C14.1, R7.1
- net $GND: now also C6.-, IC3.!EN, R17.2; no longer C17.-, C6.2, IC3.F, IC3.G, IC4.!EN, IC4.GND
- net $VCC: now also C6.+, FTDI_BASIC.4, IC3.OUT, IC3.OUT_2, IC3.SENSE/FB; no longer C17.+, IC4.OUT, IC4.OUT_2, IC4.SENSE/FB, R17.1
- net $VDD: now also IC3.IN, IC3.IN_2; no longer C6.1, IC3.VCC, IC4.IN, IC4.IN_2
- net BA0: no longer C10.1
- net BA1: now also D5.A; no longer IC3.D
- net BA2: now also D4.A; no longer IC3.C
- net BA3: now also D3.A; no longer IC3.B
- net BA4: now also D2.A; no longer IC3.H
- net BA5: now also D1.A; no longer IC3.A
- net BA6: no longer C8.1
- net BA7: no longer C7.1
- net N$16: now also IC1.P0, R1.2; no longer C9.2, IC3.X, R3.2
- net RX: no longer R17.2
- net SCL: now also R34.1; no longer R33.1
- net SDA: now also R33.1; no longer R34.1
Other:
- moved on the sheet: D1, D2, D3, ENHANCED_BUS, IC2, OSC1, R1, R10, R11, R12, R13, R14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
